File: KiCAD/MagnetPCB/MagnetPCB.kicad_sch (KiCad schematic)
At the start: 8 parts, among them J1 Screw_Terminal_01x02

Commit message: Snapshot: MagnetPCB/TMi-3 KiCAD work, journal, TouchOSC, archive Additive1
Last state of this repo before its history continues in la-harpe-eliane.
Parts:
- removed J1: Screw_Terminal_01x02, TerminalBlock_RND:TerminalBlock_RND_205-00045_1x02_P5.00mm_Horizontal, symbol Connector:Screw_Terminal_01x02
- added J1: MJ-3536NG, MJ-3536NG:CUI_MJ-3536NG, symbol MJ-3536NG:MJ-3536NG
Connections:
- net at D1.1 (K), L1.2 (+): now also J1.2
- net at D1.2 (A), H4.1, L1.1 (-): now also J1.1
Changed lines of the file:
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@@
-	(wire
-		(pts
-			(xy 151.13 115.57) (xy 151.13 118.11)
-		)
-		(stroke
-			(width 0)
-			(type default)
-		)
-	)
 	(wire
 		(pts
@@
 	(wire
 		(pts
+			(xy 161.29 110.49) (xy 161.29 111.76)
+		)
+		(stroke
+			(width 0)
+			(type default)
+		)
+	)
+	(wire
+		(pts
 			(xy 101.6 110.49) (xy 130.81 110.49)
 		)
@@
 	(wire
 		(pts
-			(xy 130.81 110.49) (xy 151.13 110.49)
+			(xy 161.29 116.84) (xy 151.13 116.84)
+		)
+		(stroke
+			(width 0)
+			(type default)
+		)
+	)
+	(wire
+		(pts
+			(xy 130.81 110.49) (xy 161.29 110.49)
+		)
+		(stroke
+			(width 0)
+			(type default)
+		)
+	)
+	(wire
+		(pts
+			(xy 151.13 116.84) (xy 151.13 118.11)
 		)
 		(stroke
@@
 			(width 0)
 			(type default)
-		)
-	)
-	(wire
-		(pts
-			(xy 151.13 113.03) (xy 151.13 110.49)
-		)
-		(stroke
-			(width 0)
-			(type default)
-		)
-	)
-	(symbol
-		(lib_id "Connector:Screw_Terminal_01x02")
-		(at 156.21 113.03 0)
-		(unit 1)
-		(body_style 1)
-		(exclude_from_sim no)
-		(in_bom yes)
-		(on_board yes)
-		(in_pos_files yes)
-		(dnp no)
-		(fields_autoplaced yes)
-		(property "Reference" "J1"
-			(at 158.75 113.0299 0)
-			(show_name no)
-			(do_not_autoplace no)
-			(effects
-				(font
-					(size 1.27 1.27)
-				)
-				(justify left)
-			)
-		)
-		(property "Value" "Screw_Terminal_01x02"
-			(at 158.75 115.5699 0)
-			(show_name no)
-			(do_not_autoplace no)
-			(effects
-				(font
-					(size 1.27 1.27)
-				)
-				(justify left)
-			)
-		)
-		(property "Footprint" "TerminalBlock_RND:TerminalBlock_RND_205-00045_1x02_P5.00mm_Horizontal"
-			(at 156.21 113.03 0)
-			(hide yes)
-			(show_name no)
-			(do_not_autoplace no)
-			(effects
-				(font
-					(size 1.27 1.27)
-				)
-			)
-		)
-		(property "Datasheet" ""
-			(at 156.21 113.03 0)
-			(hide yes)
-			(show_name no)
-			(do_not_autoplace no)
-			(effects
-				(font
-					(size 1.27 1.27)
-				)
-			)
-		)
-		(property "Description" "Generic screw terminal, single row, 01x02, script generated (kicad-library-utils/schlib/autogen/connector/)"
-			(at 156.21 113.03 0)
-			(hide yes)
-			(show_name no)
-			(do_not_autoplace no)
-			(effects
-				(font
-					(size 1.27 1.27)
-				)
-			)
-		)
-		(pin "2"
-		)
-		(pin "1"
-		)
-		(instances
-			(project "MagnetPCB"
-				(path "/e133a1ff-5a66-45b0-be81-7ac7b9efe17d"
-					(reference "J1")
-					(unit 1)
-				)
-			)
 		)
 	)
@@
 		)
 		(instances
-			(project "MagnetPCB"
+			(project "NewMagnetPCB"
 				(path "/e133a1ff-5a66-45b0-be81-7ac7b9efe17d"
 					(reference "D1")
+					(unit 1)
+				)
+			)
+		)
+	)
+	(symbol
+		(lib_id "MJ-3536NG:MJ-3536NG")
+		(at 173.99 114.3 180)
+		(unit 1)
+		(body_style 1)
+		(exclude_from_sim no)
+		(in_bom yes)
+		(on_board yes)
+		(in_pos_files yes)
+		(dnp no)
+		(fields_autoplaced yes)
+		(property "Reference" "J1"
+			(at 182.88 113.0299 0)
+			(show_name no)
+			(do_not_autoplace no)
+			(effects
+				(font
+					(size 1.27 1.27)
+				)
+				(justify right)
+			)
+		)
+		(property "Value" "MJ-3536NG"
+			(at 182.88 115.5699 0)
+			(show_name no)
+			(do_not_autoplace no)
+			(effects
+				(font
+					(size 1.27 1.27)
+				)
+				(justify right)
+			)
+		)
+		(property "Footprint" "MJ-3536NG:CUI_MJ-3536NG"
+			(at 173.99 114.3 0)
+			(hide yes)
+			(show_name no)
+			(do_not_autoplace no)
+			(effects
+				(font
+					(size 1.27 1.27)
+				)
+				(justify bottom)
+			)
+		)
+		(property "Datasheet" ""
+			(at 173.99 114.3 0)
+			(hide yes)
+			(show_name no)
+			(do_not_autoplace no)
+			(effects
+				(font
+					(size 1.27 1.27)
+				)
+			)
+		)
+		(property "Description" ""
+			(at 173.99 114.3 0)
+			(hide yes)
+			(show_name no)
+			(do_not_autoplace no)
+			(effects
+				(font
+					(size 1.27 1.27)
+				)
+			)
+		)
+		(property "PARTREV" "1.03"
+			(at 173.99 114.3 0)
+			(hide yes)
+			(show_name no)
+			(do_not_autoplace no)
+			(effects
+				(font
+					(size 1.27 1.27)
+				)
+				(justify bottom)
+			)
+		)
+		(property "STANDARD" "Manufacturer Recommendations"
+			(at 173.99 114.3 0)
+			(hide yes)
+			(show_name no)
+			(do_not_autoplace no)
+			(effects
+				(font
+					(size 1.27 1.27)
+				)
+				(justify bottom)
+			)
+		)
+		(property "MAXIMUM_PACKAGE_HEIGHT" "10.2mm"
+			(at 173.99 114.3 0)
+			(hide yes)
+			(show_name no)
+			(do_not_autoplace no)
+			(effects
+				(font
+					(size 1.27 1.27)
+				)
+				(justify bottom)
+			)
+		)
+		(property "MANUFACTURER" "Cui Devices"
+			(at 173.99 114.3 0)
+			(hide yes)
+			(show_name no)
+			(do_not_autoplace no)
+			(effects
+				(font
+					(size 1.27 1.27)
+				)
+				(justify bottom)
+			)
+		)
+		(pin "3"
+		)
+		(pin "1"
+		)
+		(pin "2"
+		)
+		(instances
+			(project "NewMagnetPCB"
+				(path "/e133a1ff-5a66-45b0-be81-7ac7b9efe17d"
+					(reference "J1")
 					(unit 1)
 				)
@@
 		)
 		(instances
-			(project "MagnetPCB"
+			(project "NewMagnetPCB"
 				(path "/e133a1ff-5a66-45b0-be81-7ac7b9efe17d"
 					(reference "H2")
@@
 		)
 		(instances
-			(project "MagnetPCB"
+			(project "NewMagnetPCB"
 				(path "/e133a1ff-5a66-45b0-be81-7ac7b9efe17d"
 					(reference "H4")
@@
 		)
 		(instances
-			(project "MagnetPCB"
+			(project "NewMagnetPCB"
 				(path "/e133a1ff-5a66-45b0-be81-7ac7b9efe17d"
 					(reference "H5")
@@
 		)
 		(instances
-			(project "MagnetPCB"
+			(project "NewMagnetPCB"
 				(path "/e133a1ff-5a66-45b0-be81-7ac7b9efe17d"
 					(reference "H3")
@@
 		)
 		(instances
-			(project "MagnetPCB"
+			(project "NewMagnetPCB"
 				(path "/e133a1ff-5a66-45b0-be81-7ac7b9efe17d"
 					(reference "L1")
@@
 		)
 		(instances
-			(project "MagnetPCB"
+			(project "NewMagnetPCB"
 				(path "/e133a1ff-5a66-45b0-be81-7ac7b9efe17d"
 					(reference "H6")
