File: KiCAD/TMi-3/TMi-3.kicad_sch (KiCad schematic)
At the start: 41 parts, among them J1 MJ-3536NG, J2 MJ-3536NG, J3 MJ-3536NG, J4 MJ-3536NG, J5 NMJ4HFD3, J6 NMJ4HFD3, J7 NMJ4HFD3, J8 NMJ4HFD3, J9 Barrel_Jack_Switch, Q1 IRLZ44N, Q2 IRLZ44N, Q3 IRLZ44N, Q4 IRLZ44N

Commit message: Snapshot: MagnetPCB/TMi-3 KiCAD work, journal, TouchOSC, archive Additive1
Last state of this repo before its history continues in la-harpe-eliane.
Parts:
- J1, J2, J3, J4: footprint Connector_Audio:MJ3536NG_Tighter_Pads -> MJ-3536NG:CUI_MJ-3536NG; MANUFACTURER (none) -> Cui Devices; MAXIMUM_PACKAGE_HEIGHT (none) -> 10.2mm; PARTREV (none) -> 1.03; STANDARD (none) -> Manufacturer Recommendations
Connections:
- net +12V: no longer J1.2, J1.3, J2.2, J2.3, J3.2, J3.3, J4.2, J4.3
- net at D8.2 (A), Q4.2 (D): no longer J4.1
- net at D2.2 (A), Q1.2 (D): no longer J1.1
- net at D6.2 (A), Q3.2 (D): no longer J3.1
- net at D4.2 (A), Q2.2 (D): no longer J2.1
